File: lightNecklace.kicad_pcb (KiCad board)
At the start: 2 copper layers, 64.6 x 22.2 mm, 75 parts, among them J1 USB_OTG, J2 CONN_02X03, U1 button, U101 JS202011JCQN, U102 TPS61240, U103 CD74HC4067SM96, U104 button, U105 button, U106 button, U107 button, U108 button, U109 button, U110 button, U111 button, U112 button, U113 button, U114 button, U115 button, U2 ATMEGA32U4RC-AU, Y1 Crystal_GND24

Commit message: Actual final
Other:
- board text removed: "You Caught me"
Changed lines of the file:
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@@
     (links 162)
     (no_connects 0)
-    (area 113.335999 74.854999 178.129001 97.230001)
+    (area 113.335999 71.515 178.152381 98.875)
     (thickness 1.6)
-    (drawings 7)
+    (drawings 6)
     (tracks 1352)
     (zones 0)
@@
       (xy 21.420666 3.81) (xy 21.420666 -11.091333) (xy 26.924 -11.091333) (xy 26.924 3.81)) (layer F.SilkS) (width 0.01))
   )
-  (gr_text "You Caught me" (at 160.655 95.25) (layer B.SilkS)
-    (effects (font (size 1.5 1.5) (thickness 0.3)) (justify mirror))
-  )
   (gr_circle (center 176 77) (end 177 77) (layer Edge.Cuts) (width 0.15))
